File: bms.kicad_pcb (KiCad board)
At the start: 2 copper layers, 252 x 136.7 mm, 214 parts, among them J1501 CONN_01X02, J1502 CONN_01X02, J201 CONN_01X02, J202 CONN_01X02, P1001 CONN_01X01, P1101 CONN_01X01, P1201 CONN_01X01, P1301 CONN_01X01, P1401 CONN_01X01, P1501 CONN_01X01, P1601 CONN_01X01, P1701 CONN_01X01, P1801 CONN_01X01, P1901 CONN_01X01, P2001 CONN_01X01, P201 CONN_01X01, P2101 CONN_01X01, P2201 CONN_01X01, P2301 CONN_01X01, P2401 CONN_01X01, P2501 CONN_01X01, P2601 CONN_01X01, P2701 CONN_01X01, P301 CONN_01X01, P401 CONN_01X01, P501 CONN_01X01, P601 CONN_01X01, P701 CONN_01X01, P801 CONN_01X01, P901 CONN_01X01, Q1001 DMP3130LQ, Q1101 DMP3130LQ, Q1201 DMP3130LQ, Q1301 DMP3130LQ, Q1401 DMP3130LQ, Q1501 NSV1C201MZ4, Q1601 DMP3130LQ, Q1701 DMP3130LQ, Q1801 DMP3130LQ, Q1901 DMP3130LQ, Q2001 DMP3130LQ, Q201 NSV1C201MZ4, Q2101 DMP3130LQ, Q2201 DMP3130LQ, Q2301 DMP3130LQ, Q2401 DMP3130LQ, Q2501 DMP3130LQ, Q2601 DMP3130LQ, Q2701 DMP3130LQ, Q301 DMP3130LQ, Q401 DMP3130LQ, Q501 DMP3130LQ, Q601 DMP3130LQ, Q701 DMP3130LQ, Q801 DMP3130LQ, Q901 DMP3130LQ, T1501 HX0068ANL, T201 HX0068ANL, U1501 LTC6804-1, U201 LTC6804-1

Commit message: Change LED and thermistors
Parts:
- removed R1515, R215: 1.2k, Resistors_SMD:R_0402
- added D1501: 1N4148X, Diodes_SMD:SOD-523, F.Cu at (145.3, -53.3)
- added D201: 1N4148X, Diodes_SMD:SOD-523, F.Cu at (143.5, 170.9)
- added LED1502: SML-P12MTT86R, LEDs:LED_0402, F.Cu at (147.7, -53.2)
- added LED202: SML-P12MTT86R, LEDs:LED_0402, F.Cu at (143.3, 172.3)
- C1501, C201: footprint Capacitors_SMD:C_0603 -> Capacitors_SMD:C_0402
- LED1501, LED201: value Led_Small -> SML-P12MTT86R; footprint LEDs:LED_0603 -> LEDs:LED_0402
- TH1501, TH1502, TH1503, TH1504, TH1505, TH201, TH202, TH203, TH204, TH205: footprint Resistors_ThroughHole:Resistor_Vertical_RM5mm -> Measurement_Points:Test_Point_2Pads
- moved R202 152.0 mm to (272.7, 92.2), turned to 90 degrees
- moved R203 138.3 mm to (274.4, 92.2), turned to 90 degrees
- moved C207 113.8 mm to (242.6, 132.4)
- moved C206 87.0 mm to (246.6, 132.7)
- moved C204 78.4 mm to (158.7, 119.6), turned to 270 degrees
- moved C201 52.1 mm to (143.3, 127.4)
- moved C208 41.3 mm to (147.3, 130.8), turned to 90 degrees
- moved R204 39.3 mm to (150.8, 144.3)
- moved R210 25.0 mm to (124.3, 176.9)
- moved R209 24.0 mm to (148.4, 144.2)
- moved R212 23.4 mm to (123.1, 187.3)
- moved R213 23.3 mm to (135.4, 187.3)
- moved R211 18.4 mm to (134.7, 177.1)
- moved R214 16.3 mm to (146.5, 168.6)
- moved C203 9.31 mm to (156.3, 131.7)
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Connections:
- R1510 pad 1: /PackB/TEMP1 -> /PackB/V-
- R1510 pad 2: /PackB/VREF2 -> /PackB/TEMP1
- R1511 pad 1: /PackB/TEMP2 -> /PackB/V-
- R1511 pad 2: /PackB/VREF2 -> /PackB/TEMP2
- R1512 pad 1: /PackB/TEMP3 -> /PackB/V-
- R1512 pad 2: /PackB/VREF2 -> /PackB/TEMP3
- R1513 pad 1: /PackB/TEMP4 -> /PackB/V-
- R1513 pad 2: /PackB/VREF2 -> /PackB/TEMP4
- R1514 pad 1: /PackB/TEMP5 -> /PackB/V-
- R1514 pad 2: /PackB/VREF2 -> /PackB/TEMP5
- R210 pad 1: /PackA/TEMP1 -> /PackA/V-
- R210 pad 2: /PackA/VREF2 -> /PackA/TEMP1
- R211 pad 1: /PackA/TEMP2 -> /PackA/V-
- R211 pad 2: /PackA/VREF2 -> /PackA/TEMP2
- R212 pad 1: /PackA/TEMP3 -> /PackA/V-
- R212 pad 2: /PackA/VREF2 -> /PackA/TEMP3
- R213 pad 1: /PackA/TEMP4 -> /PackA/V-
- R213 pad 2: /PackA/VREF2 -> /PackA/TEMP4
- R214 pad 1: /PackA/TEMP5 -> /PackA/V-
- R214 pad 2: /PackA/VREF2 -> /PackA/TEMP5
- TH1501 pad 1: /PackB/TEMP1 -> /PackB/VREF2
- TH1501 pad 2: /PackB/V- -> /PackB/TEMP1
- TH1502 pad 1: /PackB/TEMP2 -> /PackB/VREF2
- TH1502 pad 2: /PackB/V- -> /PackB/TEMP2
- TH1503 pad 1: /PackB/TEMP3 -> /PackB/VREF2
- TH1503 pad 2: /PackB/V- -> /PackB/TEMP3
- TH1504 pad 1: /PackB/TEMP4 -> /PackB/VREF2
- TH1504 pad 2: /PackB/V- -> /PackB/TEMP4
- TH1505 pad 1: /PackB/TEMP5 -> /PackB/VREF2
- TH1505 pad 2: /PackB/V- -> /PackB/TEMP5
- TH201 pad 1: /PackA/TEMP1 -> /PackA/VREF2
- TH201 pad 2: /PackA/V- -> /PackA/TEMP1
- TH202 pad 1: /PackA/TEMP2 -> /PackA/VREF2
- TH202 pad 2: /PackA/V- -> /PackA/TEMP2
- TH203 pad 1: /PackA/TEMP3 -> /PackA/VREF2
- TH203 pad 2: /PackA/V- -> /PackA/TEMP3
- TH204 pad 1: /PackA/TEMP4 -> /PackA/VREF2
- TH204 pad 2: /PackA/V- -> /PackA/TEMP4
- TH205 pad 1: /PackA/TEMP5 -> /PackA/VREF2
- TH205 pad 2: /PackA/V- -> /PackA/TEMP5
Routing:
- net /PackA/C12: track 3.60 -> 3.05 mm

Commit message: Approx placement complete
Parts:
- moved TH204 121.6 mm to (231.3, 112.0), turned to 90 degrees
- moved R302 115.5 mm to (271.1, 92.3), turned to 90 degrees
- moved R1402 100.7 mm to (50.2, 156.2), turned to 180 degrees
- moved R402 96.6 mm to (246.2, 155.8), turned to 270 degrees
- moved TH203 82.1 mm to (190.5, 137.8), turned to 90 degrees
- moved R1302 77.5 mm to (70.5, 90.3), turned to 180 degrees
- moved TH202 76.8 mm to (68.1, 136.2), turned to 90 degrees
- moved R602 69.1 mm to (209.2, 155.4), turned to 0 degrees
- moved R1202 68.9 mm to (91.4, 155.6), turned to 180 degrees
- moved TH205 68.3 mm to (108.9, 107.8), turned to 270 degrees
- moved R213 61.2 mm to (147.6, 127.3)
- moved R212 60.2 mm to (144.6, 131.1)
- moved D201 58.4 mm to (122.2, 116.5)
- moved LED201 58.4 mm to (122.5, 115.1)
- moved LED202 58.4 mm to (122.0, 117.9)
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Connections:
- LED1501 pad 1: /PackB/TEMP5 -> /PackB/TEMP1
- LED201 pad 1: /PackA/TEMP5 -> /PackA/TEMP1
- R1510 pad 2: /PackB/TEMP1 -> /PackB/TEMP5
- R1514 pad 2: /PackB/TEMP5 -> /PackB/TEMP1
- R210 pad 2: /PackA/TEMP1 -> /PackA/TEMP5
- R214 pad 2: /PackA/TEMP5 -> /PackA/TEMP1
- TH1501 pad 2: /PackB/TEMP1 -> /PackB/TEMP5
- TH1505 pad 2: /PackB/TEMP5 -> /PackB/TEMP1
- TH201 pad 2: /PackA/TEMP1 -> /PackA/TEMP5
- TH205 pad 2: /PackA/TEMP5 -> /PackA/TEMP1
Routing:
- added copper zone on B.Cu, net /PackA/V-
Other:
- outline, holes or cut-outs redrawn

Commit message: routing progress
Parts:
- moved R201 120.2 mm to (28.6, 90.2), turned to 270 degrees
- moved D201 24.6 mm to (141.1, 132.3), turned to 90 degrees
- moved LED201 24.4 mm to (142.4, 129.2), turned to 270 degrees
- moved LED202 24.3 mm to (142.4, 131.1), turned to 270 degrees
- moved Q201 7.43 mm to (146.6, 135.7), turned to 90 degrees
- moved C203 5.86 mm to (153.1, 136.6), turned to 0 degrees
- moved C208 4.64 mm to (152.0, 134.1), turned to 270 degrees
- moved R208 4.40 mm to (152.9, 131.6), turned to 180 degrees
- moved R204 2.82 mm to (157.4, 128.3), turned to 270 degrees
- moved R209 1.78 mm to (156.3, 127.4), turned to 270 degrees
- moved C1401 1.62 mm to (143.6, 122.4)
- moved C202 0.65 mm to (151.6, 129.3), turned to 270 degrees
- moved R207 0.39 mm to (151.8, 127.2), turned to 0 degrees
- moved R206 0.36 mm to (154.6, 127.5)
- moved C205 0.15 mm to (148.8, 128.6)
Connections:
- net Net-(Q1001-Pad3) renamed /PackA/Cell5/DISCH'
- net Net-(Q1101-Pad3) renamed /PackA/Cell4/DISCH'
- net Net-(Q1201-Pad3) renamed /PackA/Cell3/DISCH'
- net Net-(Q1301-Pad3) renamed /PackA/Cell2/DISCH'
- net Net-(Q1401-Pad3) renamed /PackA/Cell1/DISCH'
- net Net-(Q1601-Pad3) renamed /PackB/Cell12/DISCH'
- net Net-(Q1701-Pad3) renamed /PackB/Cell11/DISCH'
- net Net-(Q1801-Pad3) renamed /PackB/Cell10/DISCH'
- net Net-(Q1901-Pad3) renamed /PackB/Cell9/DISCH'
- net Net-(Q2001-Pad3) renamed /PackB/Cell8/DISCH'
- net Net-(Q2101-Pad3) renamed /PackB/Cell7/DISCH'
- net Net-(Q2201-Pad3) renamed /PackB/Cell6/DISCH'
- net Net-(Q2301-Pad3) renamed /PackB/Cell5/DISCH'
- net Net-(Q2401-Pad3) renamed /PackB/Cell4/DISCH'
- net Net-(Q2501-Pad3) renamed /PackB/Cell3/DISCH'
- net Net-(Q2601-Pad3) renamed /PackB/Cell2/DISCH'
- net Net-(Q2701-Pad3) renamed /PackB/Cell1/DISCH'
- net Net-(Q301-Pad3) renamed /PackA/Cell12/DISCH'
- net Net-(Q401-Pad3) renamed /PackA/Cell11/DISCH'
- net Net-(Q501-Pad3) renamed /PackA/Cell10/DISCH'
- net Net-(Q601-Pad3) renamed /PackA/Cell9/DISCH'
- net Net-(Q701-Pad3) renamed /PackA/Cell8/DISCH'
- net Net-(Q801-Pad3) renamed /PackA/Cell7/DISCH'
- net Net-(Q901-Pad3) renamed /PackA/Cell6/DISCH'
Routing:
- net /PackA/DRIVE: track 0.00 -> 16.0 mm
- net /PackA/VREG: track 0.00 -> 10.7 mm
- net /PackA/V-: track 0.00 -> 8.61 mm, vias 0 -> 12
- net /PackA/TEMP3: track 0.00 -> 6.83 mm
- net Net-(R208-Pad1): track 0.00 -> 6.36 mm
- net /PackA/C1: track 4.10 -> 10.4 mm
- net /PackA/TEMP2: track 0.00 -> 5.24 mm
- net /PackA/TEMP5: track 0.00 -> 5.21 mm
- net Net-(R204-Pad1): track 0.00 -> 4.35 mm
- net /PackA/C0: track 0.00 -> 4.08 mm
- net /PackA/VREF1: track 0.00 -> 3.63 mm
- net /PackA/TEMP1: track 0.00 -> 3.52 mm
- net /PackA/VREF2: track 0.00 -> 3.16 mm
- net Net-(R206-Pad2): track 0.00 -> 2.91 mm
- net Net-(C203-Pad1): track 0.00 -> 2.87 mm
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Other:
- net class Default: clearance 0.1778 -> 0.1524; trace_width 0.1778 -> 0.1524
- net class Discharge added: clearance 0.1524, trace_width 0.3048, via_dia 0.508, via_drill 0.254
- rule pad_to_mask_clearance: 0.14 -> 0.127
- rule trace_clearance: 0.1778 -> 0.1524
