File: bms.kicad_pcb (KiCad board)
At the start: 2 copper layers, 252 x 136.7 mm, 216 parts, among them J1501 CONN_01X02, J1502 CONN_01X02, J201 CONN_01X02, J202 CONN_01X02, P1001 CONN_01X01, P1101 CONN_01X01, P1201 CONN_01X01, P1301 CONN_01X01, P1401 CONN_01X01, P1501 CONN_01X01, P1601 CONN_01X01, P1701 CONN_01X01, P1801 CONN_01X01, P1901 CONN_01X01, P2001 CONN_01X01, P201 CONN_01X01, P2101 CONN_01X01, P2201 CONN_01X01, P2301 CONN_01X01, P2401 CONN_01X01, P2501 CONN_01X01, P2601 CONN_01X01, P2701 CONN_01X01, P301 CONN_01X01, P401 CONN_01X01, P501 CONN_01X01, P601 CONN_01X01, P701 CONN_01X01, P801 CONN_01X01, P901 CONN_01X01, Q1001 DMP3130LQ, Q1101 DMP3130LQ, Q1201 DMP3130LQ, Q1301 DMP3130LQ, Q1401 DMP3130LQ, Q1501 NSV1C201MZ4, Q1601 DMP3130LQ, Q1701 DMP3130LQ, Q1801 DMP3130LQ, Q1901 DMP3130LQ, Q2001 DMP3130LQ, Q201 NSV1C201MZ4, Q2101 DMP3130LQ, Q2201 DMP3130LQ, Q2301 DMP3130LQ, Q2401 DMP3130LQ, Q2501 DMP3130LQ, Q2601 DMP3130LQ, Q2701 DMP3130LQ, Q301 DMP3130LQ, Q401 DMP3130LQ, Q501 DMP3130LQ, Q601 DMP3130LQ, Q701 DMP3130LQ, Q801 DMP3130LQ, Q901 DMP3130LQ, T1501 HX0068ANL, T201 HX0068ANL, U1501 LTC6804-1, U201 LTC6804-1

Commit message: discharge paths routed
Parts:
- moved C207 10.7 mm to (238.8, 122.4), turned to 270 degrees
- moved C206 10.4 mm to (238.5, 126.2), turned to 180 degrees
- moved R1303 8.13 mm to (67.6, 95.2), turned to 90 degrees
- moved R402 5.33 mm to (241.0, 154.7)
- moved C201 4.37 mm to (143.5, 122.8), turned to 90 degrees
- moved R602 3.94 mm to (207.5, 151.9), turned to 270 degrees
- moved R403 3.07 mm to (241.0, 152.8)
- moved C1401 1.91 mm to (143.5, 120.5)
- moved R205 1.52 mm to (158.3, 124.6), turned to 270 degrees
- moved R601 1.28 mm to (201.9, 150.9)
- moved Q401 1.03 mm to (243.8, 153.9)
- moved R1202 0.93 mm to (92.3, 155.9)
- moved R204 0.84 mm to (157.7, 127.6)
- moved Q501 0.71 mm to (231.4, 93.1)
- moved R901 0.33 mm to (133.1, 95.4)
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Routing:
- net /PackA/Cell4/Cell+: track 0.00 -> 85.2 mm
- net /PackA/Cell9/Cell+: track 0.00 -> 82.3 mm
- net /PackA/Cell3/Cell+: track 0.00 -> 81.2 mm
- net /PackA/Cell6/Cell+: track 0.00 -> 80.6 mm
- net /PackA/V-: track 8.61 -> 86.7 mm, vias 12 -> 14
- net /PackA/Cell1/Cell+: track 0.00 -> 76.3 mm
- net /PackA/Cell5/Cell+: track 0.00 -> 74.1 mm
- net /PackA/Cell11/Cell+: track 0.00 -> 71.5 mm
- net /PackA/Cell8/Cell+: track 0.00 -> 70.8 mm
- net /PackA/Cell7/Cell+: track 0.00 -> 68.4 mm
- net /PackA/Cell2/Cell+: track 0.00 -> 64.4 mm
- net /PackA/Cell10/Cell+: track 0.00 -> 62.8 mm
- net /PackA/VREG: track 10.7 -> 20.7 mm
- net Net-(C203-Pad1): track 2.87 -> 9.47 mm
- net /PackA/Cell8/DISCH': track 0.00 -> 5.26 mm
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
Commit message: sense paths routed
Parts:
- moved R1203 1.31 mm to (77.8, 150.8)
- moved R602 0.63 mm to (207.0, 152.3), turned to 0 degrees
Routing:
- net /PackA/C0: track 6.43 -> 134.8 mm, vias 0 -> 2
- net /PackA/C12: track 3.05 -> 130.4 mm, vias 0 -> 2
- net /PackA/C11: track 4.56 -> 120.5 mm, vias 0 -> 2
- net /PackA/C1: track 8.50 -> 123.0 mm, vias 0 -> 4
- net /PackA/C2: track 3.57 -> 104.3 mm, vias 0 -> 2
- net /PackA/C9: track 4.15 -> 88.5 mm, vias 0 -> 4
- net /PackA/C3: track 4.53 -> 81.7 mm, vias 0 -> 2
- net /PackA/C4: track 3.23 -> 68.8 mm, vias 0 -> 2
- net /PackA/C10: track 3.40 -> 68.6 mm, vias 0 -> 2
- net /PackA/C7: track 3.96 -> 68.9 mm, vias 0 -> 2
- net /PackA/C5: track 4.11 -> 65.3 mm, vias 0 -> 2
- net /PackA/C8: track 3.00 -> 39.1 mm, vias 0 -> 2
- net /PackA/C6: track 2.93 -> 30.9 mm
- net /PackA/Cell10/Cell+: track 62.8 -> 86.8 mm
- net Net-(Q1201-Pad1): track 0.00 -> 20.8 mm
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
Commit message: isospi diff pairs routed
Parts:
- moved C206 1.69 mm to (240.1, 125.6), turned to 90 degrees
- moved C207 1.50 mm to (240.1, 123.1)
Routing:
- net Net-(R206-Pad1): track 2.25 -> 93.4 mm, vias 0 -> 2
- net Net-(R206-Pad2): track 2.89 -> 91.5 mm, vias 0 -> 2
- net Net-(R205-Pad1): track 3.55 -> 89.6 mm, vias 0 -> 2
- net Net-(R205-Pad2): track 1.83 -> 87.2 mm, vias 0 -> 2
Changed lines of the file:
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@@
   (general
     (links 360)
-    (no_connects 243)
+    (no_connects 230)
     (area 15.092857 -64.1644 279.107143 159.3774)
     (thickness 1.6)
     (drawings 273)
-    (tracks 645)
+    (tracks 694)
     (zones 0)
     (modules 216)
@@
   )
   (module Capacitors_SMD:C_0402 (layer F.Cu)
-    (at 238.506 126.1745 180)
+    (at 240.0935 125.603 90)
     (descr "Capacitor SMD 0402, reflow soldering, AVX (see smccp.pdf)")
     (tags "capacitor 0402")
     (attr smd)
-    (fp_text reference C206 (at 0 -1.7 180) (layer F.SilkS)
+    (fp_text reference C206 (at 0 -1.7 90) (layer F.SilkS)
       (effects (font (size 0.5 0.5) (thickness 0.11)))
     )
-    (fp_text value 100pF (at 0 1.7 180) (layer F.Fab)
+    (fp_text value 100pF (at 0 1.7 90) (layer F.Fab)
       (effects (font (size 1 1) (thickness 0.15)))
     )
@@
     (fp_line (start 0.25 -0.475) (end -0.25 -0.475) (layer F.SilkS) (width 0.15))
     (fp_line (start -0.25 0.475) (end 0.25 0.475) (layer F.SilkS) (width 0.15))
-    (pad 1 smd rect (at -0.55 0 180) (size 0.6 0.5) (layers F.Cu F.Paste F.Mask)
+    (pad 1 smd rect (at -0.55 0 90) (size 0.6 0.5) (layers F.Cu F.Paste F.Mask)
       (net 7 "Net-(C206-Pad1)"))
-    (pad 2 smd rect (at 0.55 0 180) (size 0.6 0.5) (layers F.Cu F.Paste F.Mask)
+    (pad 2 smd rect (at 0.55 0 90) (size 0.6 0.5) (layers F.Cu F.Paste F.Mask)
       (net 1 /PackA/V-))
     (model Capacitors_SMD.3dshapes/C_0402.wrl
@@
   )
   (module Capacitors_SMD:C_0402 (layer F.Cu)
-    (at 238.76 122.4495 270)
+    (at 240.0935 123.1265 270)
     (descr "Capacitor SMD 0402, reflow soldering, AVX (see smccp.pdf)")
     (tags "capacitor 0402")
@@
   (segment (start 169.06276 155.60076) (end 168.35 155.60076) (width 0.3048) (layer F.Cu) (net 56))
   (segment (start 161 150.3) (end 158.5595 147.8595) (width 0.3048) (layer F.Cu) (net 57))
-  (segment (start 159.131 128.2065) (end 159.131 124.587) (width 0.3048) (layer F.Cu) (net 57))
+  (segment (start 159.131 128.3335) (end 159.131 124.587) (width 0.3048) (layer F.Cu) (net 57))
   (segment (start 159.512 121.3485) (end 159.512 114.9985) (width 0.3048) (layer F.Cu) (net 57))
-  (segment (start 158.5595 147.8595) (end 158.5595 128.778) (width 0.3048) (layer F.Cu) (net 57))
-  (segment (start 158.5595 128.778) (end 159.131 128.2065) (width 0.3048) (layer F.Cu) (net 57))
+  (segment (start 158.5595 147.8595) (end 158.5595 128.905) (width 0.3048) (layer F.Cu) (net 57))
+  (segment (start 158.5595 128.905) (end 159.131 128.3335) (width 0.3048) (layer F.Cu) (net 57))
   (segment (start 159.131 124.587) (end 159.439301 124.278699) (width 0.3048) (layer F.Cu) (net 57))
   (segment (start 149.75 90.5045) (end 149.75 89.7) (width 0.3048) (layer F.Cu) (net 57))
@@
   (segment (start 155.5595 125.475) (end 155.5595 126.2524) (width 0.1524) (layer F.Cu) (net 101))
   (segment (start 155.5595 126.2524) (end 155.9769 126.6698) (width 0.1524) (layer F.Cu) (net 101))
+  (segment (start 240.538 120.0785) (end 241.5601 120.0785) (width 0.1524) (layer F.Cu) (net 102))
+  (segment (start 241.5601 120.0785) (end 241.7336 119.905) (width 0.1524) (layer F.Cu) (net 102))
+  (segment (start 238.062244 120.85319) (end 239.76331 120.85319) (width 0.1524) (layer B.Cu) (net 102))
+  (segment (start 239.76331 120.85319) (end 240.538 120.0785) (width 0.1524) (layer B.Cu) (net 102))
+  (via (at 240.538 120.0785) (size 0.381) (drill 0.2286) (layers F.Cu B.Cu) (net 102))
+  (segment (start 159.583995 123.58369) (end 235.331744 123.58369) (width 0.1524) (layer B.Cu) (net 102))
+  (segment (start 235.331744 123.58369) (end 238.062244 120.85319) (width 0.1524) (layer B.Cu) (net 102))
+  (segment (start 158.1785 124.3965) (end 158.368999 124.206001) (width 0.1524) (layer B.Cu) (net 102))
+  (segment (start 158.368999 124.206001) (end 158.961684 124.206001) (width 0.1524) (layer B.Cu) (net 102))
+  (segment (start 158.961684 124.206001) (end 159.583995 123.58369) (width 0.1524) (layer B.Cu) (net 102))
+  (segment (start 158.3309 123.837) (end 158.3309 124.2441) (width 0.1524) (layer F.Cu) (net 102))
+  (segment (start 158.3309 124.2441) (end 158.1785 124.3965) (width 0.1524) (layer F.Cu) (net 102))
+  (via (at 158.1785 124.3965) (size 0.381) (drill 0.2286) (layers F.Cu B.Cu) (net 102))
   (segment (start 156.6679 123.837) (end 156.0595 124.4454) (width 0.1524) (layer F.Cu) (net 102))
   (segment (start 156.0595 124.4454) (end 156.0595 125.475) (width 0.1524) (layer F.Cu) (net 102))
   (segment (start 158.3309 123.837) (end 156.6679 123.837) (width 0.1524) (layer F.Cu) (net 102))
+  (segment (start 240.4745 121.158) (end 241.7166 121.158) (width 0.1524) (layer F.Cu) (net 103))
+  (segment (start 241.7166 121.158) (end 241.7336 121.175) (width 0.1524) (layer F.Cu) (net 103))
+  (segment (start 235.458 123.8885) (end 238.1885 121.158) (width 0.1524) (layer B.Cu) (net 103))
+  (segment (start 238.1885 121.158) (end 240.4745 121.158) (width 0.1524) (layer B.Cu) (net 103))
+  (via (at 240.4745 121.158) (size 0.381) (drill 0.2286) (layers F.Cu B.Cu) (net 103))
+  (segment (start 159.710251 123.8885) (end 235.458 123.8885) (width 0.1524) (layer B.Cu) (net 103))
+  (segment (start 158.555672 124.773672) (end 158.825079 124.773672) (width 0.1524) (layer B.Cu) (net 103))
+  (segment (start 158.825079 124.773672) (end 159.710251 123.8885) (width 0.1524) (layer B.Cu) (net 103))
+  (segment (start 158.3309 125.337) (end 158.3309 124.998444) (width 0.1524) (layer F.Cu) (net 103))
+  (segment (start 158.3309 124.998444) (end 158.555672 124.773672) (width 0.1524) (layer F.Cu) (net 103))
+  (via (at 158.555672 124.773672) (size 0.381) (drill 0.2286) (layers F.Cu B.Cu) (net 103))
   (segment (start 158.3309 125.337) (end 156.6975 125.337) (width 0.1524) (layer F.Cu) (net 103))
   (segment (start 156.6975 125.337) (end 156.5595 125.475) (width 0.1524) (layer F.Cu) (net 103))
+  (segment (start 240.411 127.508) (end 241.7166 127.508) (width 0.1524) (layer F.Cu) (net 104))
+  (segment (start 241.7166 127.508) (end 241.7336 127.525) (width 0.1524) (layer F.Cu) (net 104))
+  (segment (start 158.5595 126.5555) (end 239.4585 126.5555) (width 0.1524) (layer B.Cu) (net 104))
+  (segment (start 239.4585 126.5555) (end 240.411 127.508) (width 0.1524) (layer B.Cu) (net 104))
+  (via (at 240.411 127.508) (size 0.381) (drill 0.2286) (layers F.Cu B.Cu) (net 104))
+  (segment (start 153.6693 127.4572) (end 154.0717 127.4572) (width 0.1524) (layer F.Cu) (net 104))
+  (segment (start 154.0717 127.4572) (end 155.583001 128.968501) (width 0.1524) (layer F.Cu) (net 104))
+  (segment (start 155.583001 128.968501) (end 157.897069 128.968501) (width 0.1524) (layer F.Cu) (net 104))
+  (segment (start 157.897069 128.968501) (end 158.5595 128.30607) (width 0.1524) (layer F.Cu) (net 104))
+  (segment (start 158.5595 128.30607) (end 158.5595 126.5555) (width 0.1524) (layer F.Cu) (net 104))
+  (via (at 158.5595 126.5555) (size 0.381) (drill 0.2286) (layers F.Cu B.Cu) (net 104))
   (segment (start 153.0595 125.475) (end 153.0595 126.3514) (width 0.1524) (layer F.Cu) (net 104))
   (segment (start 153.0595 126.3514) (end 153.5811 126.873) (width 0.1524) (layer F.Cu) (net 104))
   (segment (start 153.5811 126.873) (end 153.5557 127.3436) (width 0.1524) (layer F.Cu) (net 104) (status 20))
   (segment (start 153.5557 127.3436) (end 153.6693 127.4572) (width 0.1524) (layer F.Cu) (net 104) (status 30))
+  (segment (start 240.411 128.143) (end 241.063 128.795) (width 0.1524) (layer F.Cu) (net 105))
+  (segment (start 241.063 128.795) (end 241.7336 128.795) (width 0.1524) (layer F.Cu) (net 105))
+  (segment (start 239.9665 127.494566) (end 239.9665 127.6985) (width 0.1524) (layer B.Cu) (net 105))
+  (segment (start 239.9665 127.6985) (end 240.411 128.143) (width 0.1524) (layer B.Cu) (net 105))
+  (via (at 240.411 128.143) (size 0.381) (drill 0.2286) (layers F.Cu B.Cu) (net 105))
+  (segment (start 239.332244 126.86031) (end 239.9665 127.494566) (width 0.1524) (layer B.Cu) (net 105))
+  (segment (start 158.88969 126.86031) (end 239.332244 126.86031) (width 0.1524) (layer B.Cu) (net 105))
+  (segment (start 154.7495 126.619) (end 155.105101 126.974601) (width 0.1524) (layer B.Cu) (net 105))
+  (segment (start 155.105101 126.974601) (end 158.775399 126.974601) (width 0.1524) (layer B.Cu) (net 105))
+  (segment (start 158.775399 126.974601) (end 158.88969 126.86031) (width 0.1524) (layer B.Cu) (net 105))
+  (segment (start 154.3685 126.9746) (end 154.8511 127.4572) (width 0.1524) (layer F.Cu) (net 105))
+  (segment (start 154.3939 126.9746) (end 154.7495 126.619) (width 0.1524) (layer F.Cu) (net 105))
+  (segment (start 154.1399 126.746) (end 154.3685 126.9746) (width 0.1524) (layer F.Cu) (net 105))
+  (segment (start 154.3685 126.9746) (end 154.3939 126.9746) (width 0.1524) (layer F.Cu) (net 105))
+  (via (at 154.7495 126.619) (size 0.381) (drill 0.2286) (layers F.Cu B.Cu) (net 105))
   (segment (start 154.8511 127.4572) (end 155.1693 127.4572) (width 0.1524) (layer F.Cu) (net 105) (status 20))
-  (segment (start 154.1399 126.746) (end 154.8511 127.4572) (width 0.1524) (layer F.Cu) (net 105))
   (segment (start 154.0531 126.746) (end 154.1399 126.746) (width 0.1524) (layer F.Cu) (net 105))
   (segment (start 153.5595 126.2524) (end 154.0531 126.746) (width 0.1524) (layer F.Cu) (net 105))

Commit message: routuing progress
Parts:
- moved R303 3.11 mm to (269.3, 96.1), turned to 90 degrees
Routing:
- net /PackA/VREF2: track 3.16 -> 227.0 mm, vias 0 -> 9
- net Net-(C203-Pad1): track 9.47 -> 163.3 mm, vias 0 -> 4
- net /PackA/V-: track 87.9 -> 220.1 mm
- net /PackA/V+: track 1.98 -> 131.3 mm, vias 0 -> 2
- net Net-(Q501-Pad1): track 0.00 -> 1.82 mm
- net Net-(Q301-Pad1): track 0.00 -> 1.82 mm

Commit message: routuing progress
Parts:
- moved R1003 11.6 mm to (122.2, 147.3), turned to 270 degrees
Routing:
- net /PackA/S1: track 0.00 -> 131.3 mm, vias 0 -> 2
- net /PackA/S2: track 0.00 -> 97.7 mm, vias 0 -> 4
- net /PackA/TEMP4: track 2.11 -> 97.2 mm, vias 0 -> 2
- net /PackA/S3: track 0.00 -> 88.0 mm, vias 0 -> 6
- net /PackA/V-: track 220.1 -> 301.8 mm, vias 14 -> 15
- net /PackA/TEMP2: track 5.24 -> 85.2 mm, vias 0 -> 2
- net /PackA/TEMP3: track 6.83 -> 73.0 mm, vias 0 -> 2
- net /PackA/TEMP1: track 3.52 -> 64.0 mm, vias 0 -> 2
- net /PackA/S4: track 0.00 -> 59.7 mm, vias 0 -> 2
- net /PackA/S5: track 0.00 -> 54.8 mm, vias 0 -> 4
- net Net-(Q1001-Pad1): track 0.00 -> 10.5 mm
- net /PackA/Cell6/Cell+: track 80.6 -> 88.7 mm
- net Net-(Q701-Pad1): track 0.00 -> 2.41 mm
- net /PackA/Cell2/Cell+: track 64.4 -> 66.5 mm
- net /PackA/Cell7/Cell+: track 68.4 -> 70.4 mm
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Other:
- outline, holes or cut-outs redrawn

Commit message: pack A routing complete?
Parts:
- moved J201 3.10 mm to (256.2, 119.8)
- moved J202 2.86 mm to (256.2, 128.7)
Routing:
- net /PackA/S12: track 0.00 -> 137.6 mm, vias 0 -> 2
- net /PackA/S11: track 0.00 -> 113.7 mm, vias 0 -> 2
- net /PackA/S10: track 0.00 -> 102.1 mm, vias 0 -> 2
- net /PackA/S9: track 0.00 -> 85.9 mm, vias 0 -> 4
- net /PackA/S7: track 0.00 -> 65.8 mm, vias 0 -> 2
- net /PackA/S8: track 0.00 -> 64.3 mm, vias 0 -> 2
- net /PackA/S6: track 0.00 -> 25.9 mm, vias 0 -> 2
- net /PackA/C9: track 88.6 -> 93.3 mm, vias 4 -> 6
- net /PackA/C7: track 68.9 -> 73.6 mm, vias 2 -> 4
- net /isoSPI_P2P_+: track 0.00 -> 3.44 mm
- net /isoSPI_P2P_-: track 0.00 -> 3.44 mm
- net /PackA/isoSPIA-: track 0.00 -> 3.33 mm
- net /PackA/isoSPIA+: track 0.00 -> 3.32 mm
- net Net-(Q901-Pad1): track 0.00 -> 2.32 mm
- net Net-(Q1301-Pad1): track 0.00 -> 1.38 mm
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