File: bms.kicad_pcb (KiCad board)
At the start: 2 copper layers, 252 x 136.7 mm, 216 parts, among them J1501 CONN_01X02, J1502 CONN_01X02, J201 CONN_01X02, J202 CONN_01X02, P1001 CONN_01X01, P1101 CONN_01X01, P1201 CONN_01X01, P1301 CONN_01X01, P1401 CONN_01X01, P1501 CONN_01X01, P1601 CONN_01X01, P1701 CONN_01X01, P1801 CONN_01X01, P1901 CONN_01X01, P2001 CONN_01X01, P201 CONN_01X01, P2101 CONN_01X01, P2201 CONN_01X01, P2301 CONN_01X01, P2401 CONN_01X01, P2501 CONN_01X01, P2601 CONN_01X01, P2701 CONN_01X01, P301 CONN_01X01, P401 CONN_01X01, P501 CONN_01X01, P601 CONN_01X01, P701 CONN_01X01, P801 CONN_01X01, P901 CONN_01X01, Q1001 DMP3130LQ, Q1101 DMP3130LQ, Q1201 DMP3130LQ, Q1301 DMP3130LQ, Q1401 DMP3130LQ, Q1501 NSV1C201MZ4, Q1601 DMP3130LQ, Q1701 DMP3130LQ, Q1801 DMP3130LQ, Q1901 DMP3130LQ, Q2001 DMP3130LQ, Q201 NSV1C201MZ4, Q2101 DMP3130LQ, Q2201 DMP3130LQ, Q2301 DMP3130LQ, Q2401 DMP3130LQ, Q2501 DMP3130LQ, Q2601 DMP3130LQ, Q2701 DMP3130LQ, Q301 DMP3130LQ, Q401 DMP3130LQ, Q501 DMP3130LQ, Q601 DMP3130LQ, Q701 DMP3130LQ, Q801 DMP3130LQ, Q901 DMP3130LQ, T1501 HX0068ANL, T201 HX0068ANL, U1501 LTC6804-1, U201 LTC6804-1

Commit message: Clone layout to pack B
Parts:
- moved R2703 218.7 mm to (36.0, 86.2), turned to 270 degrees
- moved R2701 206.6 mm to (38.0, 79.2), turned to 90 degrees
- moved R2702 202.7 mm to (50.2, 87.8), turned to 180 degrees
- moved P2701 200.2 mm to (47.8, 88.0)
- moved Q2701 199.9 mm to (38.5, 85.7)
- moved J1502 180.9 mm to (256.2, 60.4), turned to 90 degrees
- moved R2503 173.9 mm to (77.8, 82.5), turned to 180 degrees
- moved R2501 171.5 mm to (71.7, 81.0)
- moved J1501 167.5 mm to (256.2, 51.4), turned to 90 degrees
- moved Q2501 167.3 mm to (68.0, 86.5)
- moved T1501 165.9 mm to (245.9, 56.0), turned to 90 degrees
- moved P2501 161.0 mm to (88.5, 88.0)
- moved R2502 160.8 mm to (92.3, 87.5), turned to 180 degrees
- moved R1501 154.1 mm to (28.6, 21.8), turned to 270 degrees
- moved R2103 144.8 mm to (164.6, 87.2)
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Routing:
- net /PackB/V-: track 0.00 -> 301.8 mm, vias 0 -> 15
- net /PackB/VREF2: track 0.00 -> 226.9 mm, vias 0 -> 9
- net Net-(C1503-Pad1): track 0.00 -> 163.3 mm, vias 0 -> 4
- net /PackB/S12: track 0.00 -> 137.6 mm, vias 0 -> 2
- net /PackB/C0: track 0.00 -> 134.8 mm, vias 0 -> 2
- net /PackB/S1: track 0.00 -> 131.3 mm, vias 0 -> 2
- net /PackB/V+: track 0.00 -> 131.3 mm, vias 0 -> 2
- net /PackB/C12: track 0.00 -> 130.4 mm, vias 0 -> 2
- net /PackB/C1: track 0.00 -> 123.0 mm, vias 0 -> 4
- net /PackB/C11: track 0.00 -> 120.5 mm, vias 0 -> 2
- net /PackB/S11: track 0.00 -> 113.7 mm, vias 0 -> 2
- net /PackB/C2: track 0.00 -> 104.3 mm, vias 0 -> 2
- net /PackB/S10: track 0.00 -> 102.1 mm, vias 0 -> 2
- net /PackB/TEMP4: track 0.00 -> 97.8 mm, vias 0 -> 2
- net /PackB/S2: track 0.00 -> 97.7 mm, vias 0 -> 4
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- added copper zone on B.Cu, net /PackB/V-
Other:
- board text added: "PACK A +"
- board text added: "PACK A -"
- board text added: "PACK B +"
- board text added: "PACK B -"
- board text removed: "pack +"
- board text removed: "pack -"

Commit message: Fix trace-across-cutout
Parts:
- added REF**: Fiducial_1mm_Dia_2.54mm_Outer_CopperTop, Fiducials:Fiducial_1mm_Dia_2.54mm_Outer_CopperTop, F.Cu at (156.8, 133.5)
- added REF**: Fiducial_1mm_Dia_2.54mm_Outer_CopperTop, Fiducials:Fiducial_1mm_Dia_2.54mm_Outer_CopperTop, F.Cu at (156.5, 70.9)
- added REF**: Fiducial_1mm_Dia_2.54mm_Outer_CopperTop, Fiducials:Fiducial_1mm_Dia_2.54mm_Outer_CopperTop, F.Cu at (141.2, 43.9)
- added REF**: Fiducial_1mm_Dia_2.54mm_Outer_CopperTop, Fiducials:Fiducial_1mm_Dia_2.54mm_Outer_CopperTop, F.Cu at (140.9, 113.0)
- added REF**: Fiducial_1mm_Dia_2.54mm_Outer_CopperTop, Fiducials:Fiducial_1mm_Dia_2.54mm_Outer_CopperTop, F.Cu at (29.1, 26.8)
- added REF**: Fiducial_1mm_Dia_2.54mm_Outer_CopperTop, Fiducials:Fiducial_1mm_Dia_2.54mm_Outer_CopperTop, F.Cu at (28.6, 150.6)
- added REF**: Fiducial_1mm_Dia_2.54mm_Outer_CopperTop, Fiducials:Fiducial_1mm_Dia_2.54mm_Outer_CopperTop, F.Cu at (258.0, 148.6)
Routing:
- net /isoSPI_P2P_+: track 6.77 -> 78.6 mm, vias 0 -> 2
- net /isoSPI_P2P_-: track 6.77 -> 78.3 mm, vias 0 -> 2
- net /PackA/S12: track 137.6 -> 147.0 mm
- net /PackB/S12: track 137.6 -> 145.4 mm
- net /PackA/Cell11/Cell+: track 83.0 -> 83.9 mm
- net /PackB/Cell11/Cell+: track 83.0 -> 83.6 mm, vias 0 -> 1
Other:
- outline, holes or cut-outs redrawn
- board text added: "A K"
- board text added: "LTC6804 Battery Murdering System v1.0"
- board text added: "Serial:"
